Commit message: odom

File: pluto_description/urdf/pluto.xacro (robot description, xacro)
@@ -25,9 +25,9 @@
   </material>
   <!-- Used for fixing robot to Gazebo 'base_link' -->
-  <link name="world"/>
-  <joint name="fixed" type="fixed">
+<!--  <link name="world"/>-->
+<!--  <joint name="fixed" type="fixed">
     <parent link="world"/>
-    <child link="base_link"/>
-  </joint>
+    <child link="/odom"/>
+  </joint>-->
   <!-- Base -->
   <link name="base_link">

Commit message: added pluto map and pluto 2nav pacakges

File: pluto_description/urdf/pluto.xacro (robot description, xacro)
@@ -88,3 +88,8 @@
     wheel_separation="${0.40}"
     wheel_radius="${0.08}"/>-->
+  <!-- Laser -->
+  <joint name="fixed" type="fixed">
+    <parent link="base_link"/>
+    <child link="laser"/>
+  </joint>
 </robot>

Commit message: improved navigation launch, added laser to xacro

File: pluto_description/urdf/pluto.xacro (robot description, xacro)
@@ -22,4 +22,7 @@
   </material>
   <material name="rubber">
+    <color rgba="0 0 0 1"/>
+  </material>
+  <material name="black_plastic">
     <color rgba="0 0 0 1"/>
   </material>
@@ -89,7 +92,17 @@
     wheel_radius="${0.08}"/>-->
   <!-- Laser -->
-  <joint name="fixed" type="fixed">
-    <parent link="base_link"/>
+  <joint name="laser_joint" type="fixed">
+    <parent link="level_1"/>
     <child link="laser"/>
+    <origin xyz="0 0 0.03" rpy="0 0 3.14" />
+    <axis xyz="0 1 0" />
   </joint>
+  <link name="laser">
+    <visual>
+      <geometry>
+        <cylinder length="0.06" radius="0.03"/>
+      </geometry>
+      <material name="black_plastic"/>
+    </visual>
+  </link>
 </robot>

Commit message: xacro: added realsense camera, launch: enabled pointcloud

File: pluto_description/urdf/pluto.xacro (robot description, xacro)
@@ -11,4 +11,5 @@
   <xacro:include filename="$(find pluto_description)/urdf/wheel.xacro" />
   <xacro:include filename="$(find pluto_description)/urdf/castor.xacro" />
+  <xacro:include filename="$(find realsense2_description)/urdf/_d435i.urdf.xacro" />
   <!-- Materials -->
   <material name="very_light_wood">
@@ -91,4 +92,24 @@
     wheel_separation="${0.40}"
     wheel_radius="${0.08}"/>-->
+  <!-- Roof -->
+  <joint name="roof_joint" type="fixed">
+    <parent link="base_link"/>
+    <child link="roof"/>
+    <origin xyz="0 0 0.16" rpy="0 0 0" />
+    <axis xyz="0 1 0" />
+  </joint>
+  <link name="roof">
+    <visual>
+      <geometry>
+        <cylinder length="0.012" radius="0.25"/>
+      </geometry>
+      <material name="light_wood"/>
+    </visual>
+    <collision>
+      <geometry>
+        <cylinder length="0.012" radius="0.25"/>
+      </geometry>
+    </collision>
+  </link>
   <!-- Laser -->
   <joint name="laser_joint" type="fixed">
@@ -106,3 +127,7 @@
     </visual>
   </link>
+  <!-- Camera -->
+  <xacro:sensor_d435i parent="roof" use_nominal_extrinsics="true">
+    <origin xyz="0 0 0.45" rpy="0 0.57 0"/>
+  </xacro:sensor_d435i>
 </robot>

Commit message: updated camera mount in xacro

File: pluto_description/urdf/pluto.xacro (robot description, xacro)
@@ -129,5 +129,5 @@
   <!-- Camera -->
   <xacro:sensor_d435i parent="roof" use_nominal_extrinsics="true">
-    <origin xyz="0 0 0.45" rpy="0 0.57 0"/>
+    <origin xyz="0 0 0.42" rpy="0 0.57 0"/>
   </xacro:sensor_d435i>
 </robot>

Commit message: updated nav config  and ;aunchfiles

File: pluto_description/urdf/pluto.xacro (robot description, xacro)
@@ -129,5 +129,5 @@
   <!-- Camera -->
   <xacro:sensor_d435i parent="roof" use_nominal_extrinsics="true">
-    <origin xyz="0 0 0.42" rpy="0 0.57 0"/>
+    <origin xyz="0.22 0 0.12" rpy="0 0.63 0"/>
   </xacro:sensor_d435i>
 </robot>

Commit message: updated camera mounton xacro

File: pluto_description/urdf/pluto.xacro (robot description, xacro)
@@ -129,5 +129,5 @@
   <!-- Camera -->
   <xacro:sensor_d435i parent="roof" use_nominal_extrinsics="true">
-    <origin xyz="0.22 0 0.12" rpy="0 0.63 0"/>
+    <origin xyz="0.195 0 0.12" rpy="0 0 0"/>
   </xacro:sensor_d435i>
 </robot>
